File: board/hw-BOB-ATSAMD11D.kicad_pcb (KiCad board)
At the start: 2 copper layers, 21.6 x 26.7 mm, 16 parts, among them U1 ATSAMD11D14A-SS, U2 SPX3819M5-L-3-3, X1 Conn_01x10_Male, X2 Conn_01x10_Male, X3 SWD, X4 USB_B_Micro

Commit message: WIP
Parts:
- X3: footprint device.farm:SWD -> Drake:SWD
- X4: footprint device.farm:conn_usb_B_micro_smd-2 -> Drake:conn_usb_B_micro_smd-2
Other:
- board text added: "Drake.cz"
- board text removed: "DEVICE.FARM"

Commit message: WIP
Parts:
- C1, C2, C3, C4, C5, C6: footprint Capacitor_SMD:C_0805_2012Metric_Pad1.15x1.40mm_HandSolder -> Capacitor_SMD:C_0805_2012Metric_Pad1.18x1.45mm_HandSolder
- R1, R2, R3: footprint Resistor_SMD:R_0805_2012Metric_Pad1.15x1.40mm_HandSolder -> Resistor_SMD:R_0805_2012Metric_Pad1.20x1.40mm_HandSolder
Connections:
- X4 pad 4: (no net) -> unconnected-(X4-ID)
Other:
- net class Default removed
- net class PWR removed
